File: hardware/ableton controller.kicad_pcb (KiCad board)
At the start: 2 copper layers, 276 x 144.5 mm, 78 parts, among them J1 USB_header, SW10 SW_rec, SW101 SW_m_rec, SW102 SW_m_play, SW11 SW_mute, SW12 SW_play, SW13 SW_solo, SW14 SW_rec, SW15 SW_mute, SW16 SW_play, SW17 SW_solo, SW18 SW_rec, SW19 SW_mute, SW20 SW_play, SW21 SW_solo, SW22 SW_rec, SW23 SW_mute, SW24 SW_play, SW25 SW_solo, SW26 SW_rec, SW27 SW_mute, SW28 SW_play, SW29 SW_solo, SW3 SW_mute, SW30 SW_rec, SW31 SW_mute, SW32 SW_play, SW33 SW_solo, SW34 SW_rec, SW4 SW_play, SW5 SW_solo, SW6 SW_rec, SW7 SW_mute, SW8 SW_play, SW9 SW_solo, U1 MCP23017_SO, U2 MCP23017_SO, U3 PCA9956BTWY, U4 PCA9956BTWY, U5 CD4051B, U6 CD4051B, U7 Teensy-LC_sidepins

Commit message: PCB: Rev2. REXT and RESET pullups. 5v caps. Rerouting/cleanup.
Parts:
- removed REF** (x4): MountingHole_3.2mm_M3_ISO7380_Pad, MountingHole:MountingHole_3.2mm_M3_ISO7380_Pad
- added C7: 10u, Capacitor_SMD:CP_Elec_4x4.5, F.Cu at (129.8, 90.2)
- added C8: 100n, Capacitor_SMD:C_0603_1608Metric_Pad1.08x0.95mm_HandSolder, F.Cu at (136.2, 87.5)
- added R10: 10k, Resistor_SMD:R_0603_1608Metric_Pad0.98x0.95mm_HandSolder, F.Cu at (214.5, 221.3)
- added R7: 1k, Resistor_SMD:R_0603_1608Metric_Pad0.98x0.95mm_HandSolder, F.Cu at (225.8, 117.4)
- added R8: 1k, Resistor_SMD:R_0603_1608Metric_Pad0.98x0.95mm_HandSolder, F.Cu at (226.4, 221.3)
- added R9: 10k, Resistor_SMD:R_0603_1608Metric_Pad0.98x0.95mm_HandSolder, F.Cu at (216.8, 117.4)
- C1: footprint Capacitor_SMD:CP_Elec_5x4.5 -> Capacitor_SMD:CP_Elec_4x4.5
- R2: footprint Resistor_SMD:R_0603_1608Metric -> Resistor_SMD:R_0603_1608Metric_Pad0.98x0.95mm_HandSolder
- moved C4 5.07 mm to (219.6, 117.4)
- moved R3 2.81 mm to (228.7, 117.4)
- moved C6 2.59 mm to (218.9, 221.3)
- moved C5 2.42 mm to (231.9, 192.6), turned to 90 degrees
- moved R5 1.91 mm to (230.9, 221.3)
- moved R6 1.48 mm to (213.1, 192.6), turned to 90 degrees
- moved R1 1.09 mm to (81.6, 97.9)
- moved R2 0.81 mm to (86.7, 97.9)
Connections:
- net +2V5 renamed +5V
- U3 pad 1: GND -> Net-(R7-Pad1)
- U3 pad 35: VCC -> Net-(R9-Pad2)
- U4 pad 1: GND -> Net-(R8-Pad1)
- U4 pad 35: VCC -> Net-(R10-Pad2)
Routing:
- net VCC: track 1132.4 -> 1028.0 mm
- net /LED_REC: track 170.0 -> 159.9 mm, vias 1 -> 2
- net Net-(R10-Pad2): track 0.00 -> 7.56 mm
- net Net-(R9-Pad2): track 0.00 -> 5.76 mm
- net +5V: track 675.1 -> 680.1 mm
- net /SCL: track 318.0 -> 313.4 mm
- net Net-(R6-Pad2): track 8.91 -> 6.18 mm
- net Net-(R7-Pad1): track 0.00 -> 2.28 mm
- net Net-(R3-Pad1): track 4.56 -> 6.59 mm
- net Net-(R8-Pad1): track 0.00 -> 1.98 mm
- net /SW_PLAY: track 107.0 -> 108.7 mm
- net /LED_PLAY: track 157.1 -> 155.5 mm, vias 1 -> 2
- net /SDA: track 335.2 -> 334.1 mm
- net Net-(R5-Pad1): track 5.70 -> 6.56 mm
- net /POT_UTIL_6: track 23.9 -> 23.3 mm
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Other:
- board text added: "rev 2 (8-27-21)"
- board text removed: "rev 2 (8-24-21)"

Commit message: PCB: New panel, layout cleanup, maybe some fixes too?
Parts:
- added REF**: MountingHole_3.2mm_M3_ISO14580_Pad, MountingHole:MountingHole_3.2mm_M3_ISO14580_Pad, F.Cu at (76.8, 210.2)
- added REF**: MountingHole_3.2mm_M3_ISO14580_Pad, MountingHole:MountingHole_3.2mm_M3_ISO14580_Pad, F.Cu at (312.8, 85.9)
- added REF**: MountingHole_3.2mm_M3_ISO14580_Pad, MountingHole:MountingHole_3.2mm_M3_ISO14580_Pad, F.Cu at (135.7, 95.4)
- added REF**: MountingHole_3.2mm_M3_ISO14580_Pad, MountingHole:MountingHole_3.2mm_M3_ISO14580_Pad, F.Cu at (337.9, 205.0)
- moved C1 30.1 mm to (101.0, 130.0)
- moved C2 30.0 mm to (101.8, 123.8)
- moved J1 30.0 mm to (100.9, 119.1)
- moved U7 5.35 mm to (91.1, 92.7)
- moved R2 5.15 mm to (91.0, 95.0)
- moved R1 5.15 mm to (85.8, 95.0)
- moved RV11 0.10 mm to (328.1, 161.6)
- moved RV31 0.10 mm to (267.8, 161.6)
- moved RV41 0.10 mm to (237.6, 161.6)
- moved RV51 0.10 mm to (207.4, 161.6)
- moved RV61 0.10 mm to (177.3, 161.6)
- moved RV71 0.10 mm to (147.1, 161.6)
- moved RV81 0.10 mm to (117.0, 161.6)
Routing:
- net +5V: track 680.1 -> 652.8 mm, vias 1 -> 0
- net /MUX_POT_C: track 220.8 -> 213.1 mm
- net /MUX_POT_B: track 217.8 -> 210.2 mm
- net /MUX_POT_A: track 212.6 -> 205.2 mm
- net /ADC0: track 216.2 -> 210.3 mm
- net /SW_PLAY: track 108.7 -> 113.9 mm
- net /ADC1: track 78.1 -> 73.1 mm
- net VCC: track 1028.0 -> 1023.3 mm
- net GND: track 53.2 -> 48.5 mm
- net /SCL: track 313.4 -> 310.7 mm
- net /SDA: track 334.1 -> 332.0 mm
- net /POT_FX_4: track 67.4 -> 69.1 mm
- net /POT_FX_3: track 92.2 -> 93.4 mm
- net /POT_FX_2: track 50.4 -> 51.1 mm
Other:
- board size 276 x 144.5 mm -> 269 x 145 mm
