File: hardware/panel.kicad_pcb (KiCad board)
At the start: 2 copper layers, 276.1 x 133.4 mm, 0 parts

Commit message: PCB: New panel, layout cleanup, maybe some fixes too?
Parts:
- added  : , my_footprints:Possum_Logo, B.Cu at (76.1, 221.5)
Other:
- board size 276.1 x 133.4 mm -> 279 x 155 mm
