File: hardware/ableton controller.kicad_sch (KiCad schematic)
At the start: 26 parts, among them J1 USB_header, SW101 SW_m_rec, SW102 SW_m_play, U1 MCP23017_SO, U2 MCP23017_SO, U3 PCA9956BTWY, U4 PCA9956BTWY, U5 CD4051B, U6 CD4051B, U7 Teensy-LC_sidepins

Commit message: PCB: Rev2. REXT and RESET pullups. 5v caps. Rerouting/cleanup.
Parts:
- added C7: 10u, Capacitor_SMD:CP_Elec_4x4.5, symbol Device:C_Polarized_Small_US
- added C8: 100n, Capacitor_SMD:C_0603_1608Metric_Pad1.08x0.95mm_HandSolder, symbol Device:C_Small
- added R10, R9: 10k, Resistor_SMD:R_0603_1608Metric_Pad0.98x0.95mm_HandSolder, symbol Device:R_Small_US
- added R7, R8: 1k, Resistor_SMD:R_0603_1608Metric_Pad0.98x0.95mm_HandSolder, symbol Device:R_Small_US
- C1: footprint Capacitor_SMD:CP_Elec_5x4.5 -> Capacitor_SMD:CP_Elec_4x4.5
- R2: footprint Resistor_SMD:R_0603_1608Metric -> Resistor_SMD:R_0603_1608Metric_Pad0.98x0.95mm_HandSolder
Connections:
- net GND: now also C7.2, C8.2, R7.2, R8.2; no longer U3.1 (REXT), U4.1 (REXT)
- net VCC: now also C7.1, C8.1, R10.1, R9.1; no longer U3.35 (~RESET), U4.35 (~RESET)
- net +2V5 renamed +5V
- new net: R9.2, U3.35 (~RESET)
- new net: R8.1, U4.1 (REXT)
- new net: R7.1, U3.1 (REXT)
- new net: R10.2, U4.35 (~RESET)
Other:
- note added: "04/08h"
- note added: "06/0Ch"
- note removed: "04/08h ?"
- note removed: "06/0Ch ?"
- moved on the sheet: C1, C2, J1, R3, R5

Commit message: PCB: New panel, layout cleanup, maybe some fixes too?
Changed lines of the file:
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@@
     (stroke (width 0) (type dash) (color 0 0 0 0))
   )
-  (text "04/08h" (at 182.245 118.745 0)
+  (text "04/08h" (at 185.42 90.17 0)
     (effects (font (size 1.27 1.27)) (justify left bottom))
   )
-  (text "0B/16h" (at 182.245 164.465 0)
+  (text "0B/16h" (at 186.055 154.305 0)
     (effects (font (size 1.27 1.27)) (justify left bottom))
   )
-  (text "06/0Ch" (at 252.095 118.745 0)
+  (text "06/0Ch" (at 255.905 90.17 0)
     (effects (font (size 1.27 1.27)) (justify left bottom))
   )
-  (text "0D/1Ah" (at 252.095 164.465 0)
+  (text "0D/1Ah" (at 255.905 154.94 0)
     (effects (font (size 1.27 1.27)) (justify left bottom))
   )

Commit message: PCB: Tweaks? Fixes?
Connections:
- net VCC: now also R4.2, R6.2; no longer R4.1, R6.1, U1.18 (~RESET~), U2.18 (~RESET~)
- net at U2.16 (A1), U2.17 (A2): now also R6.1, U2.18 (~RESET~); no longer R6.2
- net at U1.17 (A2): now also R4.1, U1.18 (~RESET~); no longer R4.2
Other:
- moved on the sheet: R4, R6
Changed lines of the file:
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@@
   (junction (at 161.925 160.655) (diameter 0.9144) (color 0 0 0 0))
   (junction (at 161.925 165.735) (diameter 0.9144) (color 0 0 0 0))
-  (junction (at 169.545 104.775) (diameter 0.9144) (color 0 0 0 0))
   (junction (at 169.545 122.555) (diameter 0.9144) (color 0 0 0 0))
+  (junction (at 170.815 104.775) (diameter 0.9144) (color 0 0 0 0))
   (junction (at 198.12 67.31) (diameter 0.9144) (color 0 0 0 0))
   (junction (at 208.915 198.755) (diameter 0.9144) (color 0 0 0 0))
@@
   (junction (at 231.775 157.48) (diameter 0.9144) (color 0 0 0 0))
   (junction (at 231.775 165.735) (diameter 0.9144) (color 0 0 0 0))
-  (junction (at 239.395 104.775) (diameter 0.9144) (color 0 0 0 0))
-  (junction (at 239.395 117.475) (diameter 0.9144) (color 0 0 0 0))
+  (junction (at 240.665 104.775) (diameter 0.9144) (color 0 0 0 0))
+  (junction (at 240.665 117.475) (diameter 0.9144) (color 0 0 0 0))
   (junction (at 267.97 67.31) (diameter 0.9144) (color 0 0 0 0))
   (junction (at 278.765 198.755) (diameter 0.9144) (color 0 0 0 0))
@@
     (stroke (width 0) (type solid) (color 0 0 0 0))
   )
+  (wire (pts (xy 161.925 104.775) (xy 161.925 103.505))
+    (stroke (width 0) (type solid) (color 0 0 0 0))
+  )
   (wire (pts (xy 161.925 153.035) (xy 161.925 157.48))
     (stroke (width 0) (type solid) (color 0 0 0 0))
@@
     (stroke (width 0) (type solid) (color 0 0 0 0))
   )
+  (wire (pts (xy 164.465 104.775) (xy 161.925 104.775))
+    (stroke (width 0) (type solid) (color 0 0 0 0))
+  )
   (wire (pts (xy 167.64 153.035) (xy 172.085 153.035))
     (stroke (width 0) (type solid) (color 0 0 0 0))
   )
-  (wire (pts (xy 169.545 104.775) (xy 172.085 104.775))
-    (stroke (width 0) (type solid) (color 0 0 0 0))
-  )
-  (wire (pts (xy 169.545 108.585) (xy 169.545 104.775))
-    (stroke (width 0) (type solid) (color 0 0 0 0))
-  )
-  (wire (pts (xy 169.545 117.475) (xy 169.545 113.665))
+  (wire (pts (xy 169.545 104.775) (xy 170.815 104.775))
     (stroke (width 0) (type solid) (color 0 0 0 0))
   )
@@
     (stroke (width 0) (type solid) (color 0 0 0 0))
   )
+  (wire (pts (xy 170.815 104.775) (xy 172.085 104.775))
+    (stroke (width 0) (type solid) (color 0 0 0 0))
+  )
+  (wire (pts (xy 170.815 117.475) (xy 170.815 104.775))
+    (stroke (width 0) (type solid) (color 0 0 0 0))
+  )
   (wire (pts (xy 170.815 141.605) (xy 170.815 142.875))
     (stroke (width 0) (type solid) (color 0 0 0 0))
@@
     (stroke (width 0) (type solid) (color 0 0 0 0))
   )
-  (wire (pts (xy 172.085 117.475) (xy 169.545 117.475))
+  (wire (pts (xy 172.085 117.475) (xy 170.815 117.475))
     (stroke (width 0) (type solid) (color 0 0 0 0))
   )
@@
     (stroke (width 0) (type solid) (color 0 0 0 0))
   )
+  (wire (pts (xy 231.775 104.775) (xy 231.775 103.505))
+    (stroke (width 0) (type solid) (color 0 0 0 0))
+  )
+  (wire (pts (xy 231.775 104.775) (xy 234.315 104.775))
+    (stroke (width 0) (type solid) (color 0 0 0 0))
+  )
   (wire (pts (xy 231.775 153.035) (xy 231.775 157.48))
     (stroke (width 0) (type solid) (color 0 0 0 0))
@@
     (stroke (width 0) (type solid) (color 0 0 0 0))
   )
-  (wire (pts (xy 239.395 104.775) (xy 239.395 108.585))
-    (stroke (width 0) (type solid) (color 0 0 0 0))
-  )
-  (wire (pts (xy 239.395 104.775) (xy 241.935 104.775))
-    (stroke (width 0) (type solid) (color 0 0 0 0))
-  )
-  (wire (pts (xy 239.395 117.475) (xy 239.395 113.665))
-    (stroke (width 0) (type solid) (color 0 0 0 0))
-  )
-  (wire (pts (xy 239.395 120.015) (xy 239.395 117.475))
+  (wire (pts (xy 239.395 104.775) (xy 240.665 104.775))
     (stroke (width 0) (type solid) (color 0 0 0 0))
   )
@@
     (stroke (width 0) (type solid) (color 0 0 0 0))
   )
+  (wire (pts (xy 240.665 104.775) (xy 240.665 117.475))
+    (stroke (width 0) (type solid) (color 0 0 0 0))
+  )
+  (wire (pts (xy 240.665 104.775) (xy 241.935 104.775))
+    (stroke (width 0) (type solid) (color 0 0 0 0))
+  )
+  (wire (pts (xy 240.665 120.015) (xy 240.665 117.475))
+    (stroke (width 0) (type solid) (color 0 0 0 0))
+  )
   (wire (pts (xy 240.665 141.605) (xy 240.665 142.875))
     (stroke (width 0) (type solid) (color 0 0 0 0))
@@
     (stroke (width 0) (type solid) (color 0 0 0 0))
   )
-  (wire (pts (xy 241.935 117.475) (xy 239.395 117.475))
-    (stroke (width 0) (type solid) (color 0 0 0 0))
-  )
-  (wire (pts (xy 241.935 120.015) (xy 239.395 120.015))
+  (wire (pts (xy 241.935 117.475) (xy 240.665 117.475))
+    (stroke (width 0) (type solid) (color 0 0 0 0))
+  )
+  (wire (pts (xy 241.935 120.015) (xy 240.665 120.015))
     (stroke (width 0) (type solid) (color 0 0 0 0))
   )
@@
     (pin "1")
   )
-  (symbol (lib_id "power:VCC") (at 169.545 104.775 0) (unit 1)
+  (symbol (lib_id "power:VCC") (at 161.925 103.505 0) (unit 1)
     (in_bom yes) (on_board yes)
-    (property "Reference" "#PWR0140" (id 0) (at 169.545 108.585 0)
-      (effects (font (size 1.27 1.27)) hide)
-    )
-    (property "Value" "VCC" (id 1) (at 169.545 100.965 0))
-    (property "Footprint" "" (id 2) (at 169.545 104.775 0)
-      (effects (font (size 1.27 1.27)) hide)
-    )
-    (property "Datasheet" "" (id 3) (at 169.545 104.775 0)
+    (property "Reference" "#PWR0140" (id 0) (at 161.925 107.315 0)
+      (effects (font (size 1.27 1.27)) hide)
+    )
+    (property "Value" "VCC" (id 1) (at 161.925 99.695 0))
+    (property "Footprint" "" (id 2) (at 161.925 103.505 0)
+      (effects (font (size 1.27 1.27)) hide)
+    )
+    (property "Datasheet" "" (id 3) (at 161.925 103.505 0)
       (effects (font (size 1.27 1.27)) hide)
     )
@@
     (pin "1")
   )
-  (symbol (lib_id "power:VCC") (at 239.395 104.775 0) (unit 1)
+  (symbol (lib_id "power:VCC") (at 231.775 103.505 0) (unit 1)
     (in_bom yes) (on_board yes)
-    (property "Reference" "#PWR0134" (id 0) (at 239.395 108.585 0)
-      (effects (font (size 1.27 1.27)) hide)
-    )
-    (property "Value" "VCC" (id 1) (at 239.395 100.965 0))
-    (property "Footprint" "" (id 2) (at 239.395 104.775 0)
-      (effects (font (size 1.27 1.27)) hide)
-    )
-    (property "Datasheet" "" (id 3) (at 239.395 104.775 0)
+    (property "Reference" "#PWR0134" (id 0) (at 231.775 107.315 0)
+      (effects (font (size 1.27 1.27)) hide)
+    )
+    (property "Value" "VCC" (id 1) (at 231.775 99.695 0))
+    (property "Footprint" "" (id 2) (at 231.775 103.505 0)
+      (effects (font (size 1.27 1.27)) hide)
+    )
+    (property "Datasheet" "" (id 3) (at 231.775 103.505 0)
       (effects (font (size 1.27 1.27)) hide)
     )
@@
     (pin "2")
   )
-  (symbol (lib_id "Device:R_Small_US") (at 169.545 111.125 0) (unit 1)
+  (symbol (lib_id "Device:R_Small_US") (at 167.005 104.775 270) (unit 1)
     (in_bom yes) (on_board yes)
-    (property "Reference" "R4" (id 0) (at 165.735 110.4899 0)
+    (property "Reference" "R4" (id 0) (at 167.6401 100.965 0)
       (effects (font (size 1.27 1.27)) (justify left))
     )
-    (property "Value" "10k" (id 1) (at 165.735 113.0299 0)
+    (property "Value" "10k" (id 1) (at 165.1001 100.965 0)
       (effects (font (size 1.27 1.27)) (justify left))
     )
-    (property "Footprint" "Resistor_SMD:R_0603_1608Metric_Pad0.98x0.95mm_HandSolder" (id 2) (at 169.545 111.125 0)
-      (effects (font (size 1.27 1.27)) hide)
-    )
-    (property "Datasheet" "~" (id 3) (at 169.545 111.125 0)
+    (property "Footprint" "Resistor_SMD:R_0603_1608Metric_Pad0.98x0.95mm_HandSolder" (id 2) (at 167.005 104.775 0)
+      (effects (font (size 1.27 1.27)) hide)
+    )
+    (property "Datasheet" "~" (id 3) (at 167.005 104.775 0)
       (effects (font (size 1.27 1.27)) hide)
     )
@@
     (pin "2")
   )
-  (symbol (lib_id "Device:R_Small_US") (at 239.395 111.125 0) (unit 1)
+  (symbol (lib_id "Device:R_Small_US") (at 236.855 104.775 270) (unit 1)
     (in_bom yes) (on_board yes)
-    (property "Reference" "R6" (id 0) (at 235.585 110.4899 0)
+    (property "Reference" "R6" (id 0) (at 237.4901 100.965 0)
       (effects (font (size 1.27 1.27)) (justify left))
     )
-    (property "Value" "10k" (id 1) (at 235.585 113.0299 0)
+    (property "Value" "10k" (id 1) (at 234.9501 100.965 0)
       (effects (font (size 1.27 1.27)) (justify left))
     )
-    (property "Footprint" "Resistor_SMD:R_0603_1608Metric_Pad0.98x0.95mm_HandSolder" (id 2) (at 239.395 111.125 0)
-      (effects (font (size 1.27 1.27)) hide)
-    )
-    (property "Datasheet" "~" (id 3) (at 239.395 111.125 0)
-      (effects (font (size 1.27 1.27)) hide)
-    )
+    (property "Footprint" "Resistor_SMD:R_0603_1608Metric_Pad0.98x0.95mm_HandSolder" (id 2) (at 236.855 104.775 0)
+      (effects (font (size 1.27 1.27)) hide)
+    )
+    (property "Datasheet" "~" (id 3) (at 236.855 104.775 0)
+      (effects (font (size 1.27 1.27)) hide)
+    )
